Commit message: video9

File: src/articubot_one/description/lidar.xacro (robot description, xacro)
@@ -4,5 +4,5 @@
         <parent link="chassis" />
         <child link="laser_frame" />
-        <origin xyz="0-1 0 0.175" rpy="0 0 0" />
+        <origin xyz="0.1 0 0.175" rpy="0 0 0" />
         <axis xyz="0 0 1" />
     </joint>
@@ -23,6 +23,33 @@
         </xacro:inertial_cylinder>
     </link>
-    <gazebo reference="laser_frame" >
+     <gazebo reference="laser_frame" >
         <material>Gazebo/Red</material>
-    </gazebo >
+        <sensor name="laser" type="ray">
+            <pose>0 0 0 0 0 0</pose>
+            <visualize>false</visualize>
+            <update_rate>10</update_rate>
+            <ray>
+                <scan>
+                    <horizontal>
+                        <samples>300</samples>
+                        <resolution>1</resolution>
+                        <min_angle>-3.14</min_angle>
+                        <max_angle>3.14</max_angle>
+                    </horizontal>
+                </scan>
+                <range>
+                    <min>0.3</min>
+                    <max>12</max>
+                    <resolution>0.01</resolution>
+                </range>
+            </ray>
+            <plugin name="laser_controller" filename="libgazebo_ros_ray_sensor.so" >
+                <ros>
+                    <argument>~/out:=scan</argument>
+                </ros>
+                <output_type>sensor_msgs/LaserScan</output_type>
+                <frame_name>laser_frame</frame_name>
+            </plugin>
+        </sensor>
+    </gazebo>
 </robot>

File: src/articubot_one/description/robot_core.xacro (robot description, xacro)
@@ -13,4 +13,7 @@
     <material name="black" >
         <color rgba="0 0 0 1" />
+    </material>
+    <material name="red" >
+        <color rgba="1 0 0 1" />
     </material>
     <link name="base_link" >
